File: PCB/eye/eye.kicad_pcb (KiCad board)
At the start: 2 copper layers, 40 x 44 mm, 49 parts, among them J1 LH128, J2 Conn_01x04, J3 Conn_01x08, J4 Conn_01x08, Q1 AO3400A, U1 RP2040, U2 W25Q32JVSS, U3 AP2112K-3.3, Y1 12MHz

Commit message: BOM + improvements
Parts:
- added D2: RED_LED, LED_SMD:LED_0603_1608Metric, B.Cu at (109.3, 95.1)
- added D3: RED_LED, LED_SMD:LED_0603_1608Metric, B.Cu at (114.4, 83.3)
- added R10: 1k, Resistor_SMD:R_0603_1608Metric, B.Cu at (110.8, 92.0)
- added R11: 1k, Resistor_SMD:R_0603_1608Metric, B.Cu at (117.5, 83.3)
- added R9: 1k, Resistor_SMD:R_0603_1608Metric, B.Cu at (109.3, 92.0)
- D1: value LED -> RED_LED
Routing:
- net +5V: track 52.3 -> 60.2 mm
- net GND: track 235.1 -> 239.5 mm
- net +3.3V: track 154.5 -> 157.7 mm
- net Net-(R10-Pad2): track 0.00 -> 1.50 mm
- net Net-(D3-K): track 0.00 -> 1.49 mm
- net Net-(D2-K): track 0.00 -> 1.49 mm
