File: PCB/eye/eye.kicad_sch (KiCad schematic)
At the start: 7 parts, among them J1 LH128, SW1 SW_Push, U1 RP2040, U2 W25Q32JVSS

Commit message: continue with rp2040
Parts:
- added C1: 0.1uF, Capacitor_SMD:C_0603_1608Metric, symbol Device:C
- added Y1: Crystal_GND24, Crystal:Crystal_SMD_0603-4Pin_6.0x3.5mm, symbol Device:Crystal_GND24
Connections:
- net +3.3V: now also C1.1
- net GND: now also C1.2
- new net: Y1.2 (G), Y1.4 (G)
Other:
- moved on the sheet: U2

Commit message: finish schematic
Parts:
- added C10, C11, C12, C13, C14, C15, C8, C9: 0.1uF, Capacitor_SMD:C_0603_1608Metric, symbol Device:C
- added C16, C17, C18: 1uF, Capacitor_SMD:C_0603_1608Metric, symbol Device:C
- added C2, C3: 33pF, Capacitor_SMD:C_0603_1608Metric, symbol Device:C
- added C4, C5, C6, C7: 10uF, Capacitor_SMD:C_0805_2012Metric, symbol Device:C
- added D1: LED, LED_SMD:LED_0603_1608Metric, symbol Device:LED
- added J2: Conn_01x04, Connector_JST:JST_XH_B4B-XH-A_1x04_P2.50mm_Vertical, symbol Connector_Generic:Conn_01x04
- added J3: Conn_01x08, Connector_PinSocket_2.54mm:PinSocket_1x08_P2.54mm_Vertical, symbol Connector_Generic:Conn_01x08
- added JP1: SolderJumper_2_Open, Jumper:SolderJumper-2_P1.3mm_Open_TrianglePad1.0x1.5mm, symbol Jumper:SolderJumper_2_Open
- added Q1: AO3400A, Package_TO_SOT_SMD:SOT-23, symbol Transistor_FET:AO3400A
- added R4: 10k, Resistor_SMD:R_0603_1608Metric, symbol Device:R
- added R5: 100k, Resistor_SMD:R_0603_1608Metric, symbol Device:R
- added R6: 22, Resistor_SMD:R_0603_1608Metric, symbol Device:R
- added R7: 100, Resistor_SMD:R_0603_1608Metric, symbol Device:R
- added R8: 1k, Resistor_SMD:R_0603_1608Metric, symbol Device:R
- added SW2: SW_Push, symbol Switch:SW_Push
- added TP1, TP10, TP2, TP3, TP4, TP5, TP6, TP7, TP8, TP9: TestPoint, TestPoint:TestPoint_Pad_D1.0mm, symbol Connector:TestPoint
- added U3: AP2112K-3.3, Package_TO_SOT_SMD:SOT-23-5, symbol Regulator_Linear:AP2112K-3.3
- R1: value 2 -> 100
- Y1: value Crystal_GND24 -> 12MHz
Connections:
- net RES is gone; now on net RST: J1.11 (Pin_11)
- net +1V1: now also C14.2, C15.2, C18.2
- net +3.3V: now also C10.2, C11.2, C12.2, C13.2, C16.2, C17.2, C5.2, C7.2, C8.2, C9.2, JP1.1 (A), R4.2, R7.2, U3.5 (VOUT)
- net CS: now also U1.28 (GPIO17)
- net DC: now also U1.31 (GPIO20)
- net GND: now also Y1.2 (G), Y1.4 (G), C10.1, C11.1, C12.1, C13.1, C14.1, C15.1, C16.1, C17.1, C18.1, C2.1, C3.1, C4.1, C5.1, C6.1, C7.1, C8.1, C9.1, J2.4 (Pin_4), J3.3 (Pin_3), Q1.2 (S), R5.1, R8.1, SW2.1, U3.2 (GND); no longer R1.1
- net SCL: now also U1.7 (GPIO5), J2.3 (Pin_3); no longer J1.9 (Pin_9)
- net SDA: now also U1.6 (GPIO4), J2.2 (Pin_2); no longer J1.10 (Pin_10)
- net at R1.2: now also Q1.1 (G), R5.2; no longer J1.2 (Pin_2)
- net at U1.11 (GPIO8): now also TP3.1
- net at U1.12 (GPIO9): now also TP4.1
- net at U1.13 (GPIO10): now also TP5.1
- net at U1.14 (GPIO11): now also TP6.1
- net at U1.15 (GPIO12): now also TP7.1
- net at U1.16 (GPIO13): now also TP8.1
- net at U1.17 (GPIO14): now also TP9.1
- net at U1.18 (GPIO15): now also TP10.1
- net TX: now reaches U1.2 (GPIO0)
- net TX: now also J3.7 (Pin_7)
- net at U1.20 (XIN): now also Y1.3, C3.2
- net at U1.21 (XOUT): now also Y1.1, C2.2
- net SWCLK: now reaches U1.24 (SWCLK)
- net SWCLK: now also J3.5 (Pin_5)
- net SWDIO: now reaches U1.25 (SWDIO)
- net SWDIO: now also J3.4 (Pin_4)
- net RUN: now reaches U1.26 (RUN)
- net RUN: now also J3.6 (Pin_6), R4.1, SW2.2
- net SCK: now reaches U1.29 (GPIO18)
- net SCK: now also J1.9 (Pin_9)
- net RX: now reaches U1.3 (GPIO1)
- net RX: now also J3.8 (Pin_8)
- net MOSI: now reaches U1.30 (GPIO19)
- net MOSI: now also J1.10 (Pin_10)
- net RST: now reaches U1.32 (GPIO21)
- net BL_PIN: now reaches U1.34 (GPIO22)
- net BL_PIN: now also R1.1
- net at U1.4 (GPIO2): now also D1.2 (A)
- net at U1.8 (GPIO6): now also TP1.1
- net at U1.9 (GPIO7): now also TP2.1
- new net: Q1.3 (D), R6.1
- new net: D1.1 (K), R8.2
- new net: J3.2 (Pin_2), JP1.2 (B), R7.1
- new net +5V: C4.2, C6.2, J2.1 (Pin_1), J3.1 (Pin_1), U3.1 (VIN), U3.3 (EN)
- new net BL: J1.2 (Pin_2), R6.2
Other:
- moved on the sheet: Y1

Commit message: add buttons
Parts:
- SW1, SW2: footprint (none) -> Button_Switch_SMD:SW_SPST_TS-1088-xR025
Changed lines of the file:
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@@
 			)
 		)
-		(property "Footprint" ""
+		(property "Footprint" "Button_Switch_SMD:SW_SPST_TS-1088-xR025"
 			(at 57.15 93.98 0)
 			(hide yes)
@@
 			)
 		)
-		(property "Footprint" ""
+		(property "Footprint" "Button_Switch_SMD:SW_SPST_TS-1088-xR025"
 			(at 55.88 83.82 0)
 			(hide yes)

Commit message: finish placement
Parts:
- added J4: Conn_01x08, Connector_PinHeader_2.54mm:PinHeader_2x04_P2.54mm_Vertical, symbol Connector_Generic:Conn_01x08
- J3: footprint Connector_PinSocket_2.54mm:PinSocket_1x08_P2.54mm_Vertical -> Connector_PinHeader_2.54mm:PinHeader_2x04_P2.54mm_Vertical
- Y1: footprint Crystal:Crystal_SMD_0603-4Pin_6.0x3.5mm -> Crystal:Crystal_SMD_3225-4Pin_3.2x2.5mm
- renumbered TP5 to G10, TP6 to G11, TP7 to G12, TP8 to G13, TP9 to G14, TP10 to G15, TP1 to G6, TP2 to G7, TP3 to G8, TP4 to G9
Connections:
- net +3.3V: now also J4.1 (Pin_1)
- net BL: now also J4.3 (Pin_3)
- net CS: now also J4.5 (Pin_5)
- net DC: now also J4.4 (Pin_4)
- net GND: now also J4.2 (Pin_2)
- net MOSI: now also J4.7 (Pin_7)
- net RST: now also J4.8 (Pin_8)
- net SCK: now also J4.6 (Pin_6)
- no-connect marks 2 -> 11

Commit message: finish Eye PCB
Parts:
- renumbered SW1 to BOOT1, SW2 to RUN1
Changed lines of the file:
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@@
 		(dnp no)
 		(fields_autoplaced yes)
-		(property "Reference" "SW1"
+		(property "Reference" "BOOT1"
 			(at 57.15 91.44 0)
 			(show_name no)
@@
 			(project "eye"
 				(path "/43a36e01-9c03-487f-b76f-d3e0c5ffafba"
-					(reference "SW1")
+					(reference "BOOT1")
 					(unit 1)
 				)
@@
 		(dnp no)
 		(fields_autoplaced yes)
-		(property "Reference" "SW2"
+		(property "Reference" "RUN1"
 			(at 55.88 81.28 0)
 			(show_name no)
@@
 			(project "eye"
 				(path "/43a36e01-9c03-487f-b76f-d3e0c5ffafba"
-					(reference "SW2")
+					(reference "RUN1")
 					(unit 1)
 				)

Commit message: BOM + improvements
Parts:
- added D2, D3: RED_LED, LED_SMD:LED_0603_1608Metric, symbol Device:LED
- added R10, R11, R9: 1k, Resistor_SMD:R_0603_1608Metric, symbol Device:R
- BOOT1, RUN1: LCSC Part (none) -> C720477
- D1: value LED -> RED_LED; LCSC Part (none) -> C19171390
- G10, G11, G12, G13, G14, G15, G6, G7, G8, G9: now left out of the parts list
- J2: LCSC Part (none) -> C144395
- J3, J4: LCSC Part (none) -> C5383105
- R6: value 22 -> 22R
- R7: value 100 -> 100R
- U1: LCSC Part (none) -> C2040
- Y1: LCSC Part (none) -> C9002
Connections:
- net +3.3V: now also D3.2 (A)
- net +5V: now also D2.2 (A)
- net GND: now also R10.1, R11.1
- new net: R10.2, R9.1
- new net: D2.1 (K), R9.2
- new net: D3.1 (K), R11.2
Other:
- moved on the sheet: C10, C11, C12, C13, C16, C8, C9

Commit message: unify BOM
Parts:
- C2, C3: LCSC Part (none) -> C1663
Changed lines of the file:
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@@
 			)
 		)
+		(property "LCSC Part" "C1663"
+			(at 58.42 138.43 90)
+			(hide yes)
+			(show_name no)
+			(do_not_autoplace no)
+			(effects
+				(font
+					(size 1.27 1.27)
+				)
+			)
+		)
 		(pin "1"
 		)
@@
 			(hide yes)
 			(show_name no)
+			(do_not_autoplace no)
+			(effects
+				(font
+					(size 1.27 1.27)
+				)
+			)
+		)
+		(property "LCSC Part" "C1663"
+			(at 58.42 125.73 90)
+			(hide yes)
+			(show_name no)
