File: PCB/mouth/mouth.kicad_pcb (KiCad board)
At the start: 2 copper layers, 0 parts

Commit message: start placing Mouth PCB components
Parts:
- added BOOT1: SW_Push, Button_Switch_SMD:SW_SPST_TS-1088-xR025, F.Cu at (194.6, 87.0)
- added C1: 0.1uF, Capacitor_SMD:C_0603_1608Metric, F.Cu at (163.4, 55.8)
- added C10: 0.1uF, Capacitor_SMD:C_0603_1608Metric, F.Cu at (163.4, 68.4)
- added C11: 0.1uF, Capacitor_SMD:C_0603_1608Metric, F.Cu at (163.4, 70.9)
- added C12: 0.1uF, Capacitor_SMD:C_0603_1608Metric, F.Cu at (163.4, 73.4)
- added C13: 0.1uF, Capacitor_SMD:C_0603_1608Metric, F.Cu at (163.4, 75.9)
- added C14: 0.1uF, Capacitor_SMD:C_0603_1608Metric, F.Cu at (144.7, 78.8)
- added C15: 0.1uF, Capacitor_SMD:C_0603_1608Metric, F.Cu at (144.7, 81.3)
- added C16: 1uF, Capacitor_SMD:C_0603_1608Metric, F.Cu at (167.4, 60.9)
- added C17: 1uF, Capacitor_SMD:C_0603_1608Metric, F.Cu at (59.9, 106.9)
- added C18: 1uF, Capacitor_SMD:C_0603_1608Metric, F.Cu at (152.8, 81.5)
- added C19: 0.1uF, Capacitor_SMD:C_0603_1608Metric, F.Cu at (59.9, 108.5)
- added C2: 33pF, Capacitor_SMD:C_0603_1608Metric, F.Cu at (163.4, 58.3)
- added C20: 0.1uF, Capacitor_SMD:C_0603_1608Metric, F.Cu at (59.9, 125.3)
- added C21: 1uF, Capacitor_SMD:C_0603_1608Metric, F.Cu at (59.9, 126.9)
- added C22: 10uF, Capacitor_SMD:C_0805_2012Metric, F.Cu at (59.9, 128.7)
- added C3: 33pF, Capacitor_SMD:C_0603_1608Metric, F.Cu at (163.4, 60.9)
- added C4: 10uF, Capacitor_SMD:C_0805_2012Metric, F.Cu at (54.9, 91.8)
- added C5: 10uF, Capacitor_SMD:C_0805_2012Metric, F.Cu at (46.6, 97.6)
- added C6: 10uF, Capacitor_SMD:C_0805_2012Metric, F.Cu at (53.4, 96.8)
- added C7: 10uF, Capacitor_SMD:C_0805_2012Metric, F.Cu at (59.9, 104.9)
- added C8: 0.1uF, Capacitor_SMD:C_0603_1608Metric, F.Cu at (163.4, 63.4)
- added C9: 0.1uF, Capacitor_SMD:C_0603_1608Metric, F.Cu at (163.4, 65.9)
- added D1: RED_LED, LED_SMD:LED_0603_1608Metric, F.Cu at (200.2, 87.8)
- added D2: RED_LED, LED_SMD:LED_0603_1608Metric, F.Cu at (54.9, 94.0)
- added D3: RED_LED, LED_SMD:LED_0603_1608Metric, F.Cu at (50.6, 101.8)
- added J1: Screw_Terminal_01x02, TerminalBlock_Phoenix:TerminalBlock_Phoenix_PT-1,5-2-5.0-H_1x02_P5.00mm_Horizontal, F.Cu at (35.4, 87.4)
- added J2: Conn_01x04, Connector_JST:JST_XH_B4B-XH-A_1x04_P2.50mm_Vertical, F.Cu at (54.2, 87.6)
- added J3: Conn_01x08, Connector_PinHeader_2.54mm:PinHeader_2x04_P2.54mm_Vertical, F.Cu at (64.5, 87.8)
- added J5: Conn_02x08_Odd_Even, Connector_PinSocket_2.54mm:PinSocket_2x08_P2.54mm_Vertical, B.Cu at (44.5, 108.0)
- added JP1: SolderJumper_2_Open, Jumper:SolderJumper-2_P1.3mm_Open_TrianglePad1.0x1.5mm, F.Cu at (65.0, 94.6)
- added R10: 1k, Resistor_SMD:R_0603_1608Metric, F.Cu at (60.1, 91.4)
- added R11: 1k, Resistor_SMD:R_0603_1608Metric, F.Cu at (47.2, 101.8)
- added R13: 22R, Resistor_SMD:R_0603_1608Metric, F.Cu at (65.9, 112.1)
- added R14: 22R, Resistor_SMD:R_0603_1608Metric, F.Cu at (65.9, 110.3)
- added R15: 22R, Resistor_SMD:R_0603_1608Metric, F.Cu at (65.9, 113.9)
- added R16: 22R, Resistor_SMD:R_0603_1608Metric, F.Cu at (65.9, 115.7)
- added R17: 22R, Resistor_SMD:R_0603_1608Metric, F.Cu at (53.9, 110.4)
- added R18: 22R, Resistor_SMD:R_0603_1608Metric, F.Cu at (53.9, 112.1)
- added R19: 22R, Resistor_SMD:R_0603_1608Metric, F.Cu at (53.9, 113.9)
- added R2: 10k, Resistor_SMD:R_0603_1608Metric, F.Cu at (167.4, 75.9)
- added R20: 22R, Resistor_SMD:R_0603_1608Metric, F.Cu at (53.9, 115.7)
- added R21: 22R, Resistor_SMD:R_0603_1608Metric, F.Cu at (53.9, 123.5)
- added R22: 22R, Resistor_SMD:R_0603_1608Metric, F.Cu at (53.9, 121.7)
- added R23: 22R, Resistor_SMD:R_0603_1608Metric, F.Cu at (53.9, 119.9)
- added R24: 22R, Resistor_SMD:R_0603_1608Metric, F.Cu at (53.9, 118.1)
- added R25: 22R, Resistor_SMD:R_0603_1608Metric, F.Cu at (65.9, 123.6)
- added R26: 22R, Resistor_SMD:R_0603_1608Metric, F.Cu at (65.9, 121.9)
- added R3: 1k, Resistor_SMD:R_0603_1608Metric, F.Cu at (171.4, 55.8)
- added R4: 10k, Resistor_SMD:R_0603_1608Metric, F.Cu at (171.4, 58.3)
- added R5: 10k, Resistor_SMD:R_0603_1608Metric, F.Cu at (171.4, 60.9)
- added R7: 100R, Resistor_SMD:R_0603_1608Metric, F.Cu at (65.0, 97.0)
- added R8: 1k, Resistor_SMD:R_0603_1608Metric, F.Cu at (171.4, 65.9)
- added R9: 1k, Resistor_SMD:R_0603_1608Metric, F.Cu at (58.3, 91.4)
- added RUN1: SW_Push, Button_Switch_SMD:SW_SPST_TS-1088-xR025, F.Cu at (194.6, 92.4)
- added U1: RP2040, Package_DFN_QFN:QFN-56-1EP_7x7mm_P0.4mm_EP3.2x3.2mm, F.Cu at (186.4, 89.4)
- added U2: W25Q32JVSS, Package_SO:SOIC-8_5.3x5.3mm_P1.27mm, F.Cu at (186.4, 80.4)
- added U3: AP2112K-3.3, Package_TO_SOT_SMD:SOT-23-5, F.Cu at (50.1, 95.5)
- added U4: 74AHCT244, Package_SO:SSOP-20_4.4x6.5mm_P0.65mm, F.Cu at (59.9, 112.9)
- added U5: 74AHCT244, Package_SO:SSOP-20_4.4x6.5mm_P0.65mm, F.Cu at (59.9, 120.9)
- added Y1: 12MHz, Crystal:Crystal_SMD_3225-4Pin_3.2x2.5mm, F.Cu at (164.0, 91.6)
Other:
- board outline added: 60 x 50 mm
- board text added: "R1"
