File: PCB/mouth/mouth.kicad_sch (KiCad schematic)
At the start: 54 parts, among them J1 LH128, J2 Conn_01x04, J3 Conn_01x08, J4 Conn_01x08, Q1 AO3400A, U1 RP2040, U2 W25Q32JVSS, U3 AP2112K-3.3, Y1 12MHz

Commit message: continue on mouth PCB
Parts:
- removed G10, G11, G12, G13, G14, G15, G6, G7, G8, G9: TestPoint, TestPoint:TestPoint_Pad_D1.0mm, symbol Connector:TestPoint
- removed J1: LH128, Extra:LH128R, symbol Connector_Generic:Conn_01x12
- removed J4: Conn_01x08, Connector_PinHeader_2.54mm:PinHeader_2x04_P2.54mm_Vertical, symbol Connector_Generic:Conn_01x08
- removed Q1: AO3400A, Package_TO_SOT_SMD:SOT-23, symbol Transistor_FET:AO3400A
- removed R1: 100, Resistor_SMD:R_0603_1608Metric, symbol Device:R
- removed R6: 22R, Resistor_SMD:R_0603_1608Metric, symbol Device:R
- added C19, C20: 0.1uF, Capacitor_SMD:C_0603_1608Metric, symbol Device:C
- added C21: 1uF, Capacitor_SMD:C_0603_1608Metric, symbol Device:C
- added C22: 10uF, Capacitor_SMD:C_0805_2012Metric, symbol Device:C
- added J1: Screw_Terminal_01x02, TerminalBlock_Phoenix:TerminalBlock_Phoenix_PT-1,5-2-5.0-H_1x02_P5.00mm_Horizontal, symbol Connector:Screw_Terminal_01x02
- added J5: Conn_02x08_Odd_Even, Connector_PinHeader_2.54mm:PinHeader_2x08_P2.54mm_Vertical, symbol Connector_Generic:Conn_02x08_Odd_Even
- added R13, R14, R15, R16, R17, R18, R19, R20, R21, R22, R23, R24, R25, R26: 22R, Resistor_SMD:R_0603_1608Metric, symbol Device:R
- added U4, U5: 74AHCT244, Package_SO:SSOP-20_4.4x6.5mm_P0.65mm, symbol 74xx:74AHCT244
- R5: value 100k -> 10k
Connections:
- net +3.3V: now also C19.2, C20.2, C21.2, C22.2
- net +5V: now also R5.2, J1.1 (Pin_1), U4.20 (VCC), U5.20 (VCC)
- net GND: now also C19.1, C20.1, C21.1, C22.1, J1.2 (Pin_2), J5.16 (Pin_16), J5.4 (Pin_4), U4.1 (1OE), U4.10 (GND), U4.19 (2OE), U5.1 (1OE), U5.10 (GND), U5.11 (2A3), U5.13 (2A2), U5.19 (2OE); no longer R5.1
- net PIN_C: now reaches U1.18 (GPIO15)
- net PIN_C: now also U5.2 (1A0)
- net PIN_R2: now reaches U1.12 (GPIO9)
- net PIN_R2: now also U4.8 (1A3)
- net PIN_G1: now reaches U1.9 (GPIO7)
- net PIN_G1: now also U4.4 (1A1)
- net PIN_E: now reaches U1.15 (GPIO12)
- net PIN_E: now also U5.6 (1A2)
- net PIN_B2: now reaches U1.14 (GPIO11)
- net PIN_B2: now also U4.15 (2A1)
- net PIN_B1: now reaches U1.11 (GPIO8)
- net PIN_B1: now also U4.6 (1A2)
- net PIN_R1: now reaches U1.8 (GPIO6)
- net PIN_R1: now also U4.2 (1A0)
- net PIN_G2: now reaches U1.13 (GPIO10)
- net PIN_G2: now also U4.17 (2A0)
- net PIN_A: now reaches U1.16 (GPIO13)
- net PIN_A: now also U4.13 (2A2)
- net PIN_B: now reaches U1.17 (GPIO14)
- net PIN_B: now also U4.11 (2A3)
- net PIN_D: now reaches U1.27 (GPIO16)
- net PIN_D: now also U5.4 (1A1)
- net BL_PIN: no longer names the net of U1.34 (GPIO22)
- net CS renamed PIN_CLK
- net PIN_CLK: now also U5.8 (1A3)
- net DC: no longer names the net of U1.31 (GPIO20)
- net MOSI renamed PIN_OE
- net PIN_OE: now also U5.15 (2A1)
- net RST: no longer names the net of U1.32 (GPIO21)
- net SCK renamed PIN_LAT
- net PIN_LAT: now also U5.17 (2A0)
- new net: R18.2, U4.5 (2Y1)
- new net: R26.2, U5.5 (2Y1)
- new net: R20.2, U4.9 (2Y3)
- new net: R24.2, U5.12 (1Y3)
- new net: R23.2, U5.14 (1Y2)
- new net: R22.2, U5.16 (1Y1)
- new net: R21.2, U5.18 (1Y0)
- new net: R25.2, U5.3 (2Y0)
- new net: R15.2, U4.14 (1Y2)
- new net: R19.2, U4.7 (2Y2)
- new net: R17.2, U4.3 (2Y0)
- new net: R16.2, U4.12 (1Y3)
- new net: R13.2, U4.16 (1Y1)
- new net: R14.2, U4.18 (1Y0)
- new net A: J5.9 (Pin_9), R19.1
- new net B: J5.10 (Pin_10), R20.1
- new net B1: J5.3 (Pin_3), R15.1
- new net B2: J5.7 (Pin_7), R18.1
- new net C: J5.11 (Pin_11), R21.1
- new net CLK: J5.13 (Pin_13), R24.1
- new net D: J5.12 (Pin_12), R22.1
- new net E: J5.8 (Pin_8), R23.1
- new net G1: J5.2 (Pin_2), R13.1
- new net G2: J5.6 (Pin_6), R17.1
- new net LAT: J5.14 (Pin_14), R25.1
- new net OE: J5.15 (Pin_15), R26.1, R5.1
- new net R1: J5.1 (Pin_1), R14.1
- new net R2: J5.5 (Pin_5), R16.1
- no-connect marks 11 -> 12
Other:
- moved on the sheet: C17, C7

Commit message: start placing Mouth PCB components
Parts:
- J5: footprint Connector_PinHeader_2.54mm:PinHeader_2x08_P2.54mm_Vertical -> Connector_PinSocket_2.54mm:PinSocket_2x08_P2.54mm_Vertical
Connections:
- net +3.3V: no longer C17.2, C19.2, C20.2, C21.2, C22.2, C7.2
- net +5V: now also C17.2, C19.2, C20.2, C21.2, C22.2, C7.2
Changed lines of the file:
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@@
 	)
 	(junction
-		(at 213.36 24.13)
-		(diameter 0)
-		(color 0 0 0 0)
-	)
-	(junction
 		(at 205.74 31.75)
 		(diameter 0)
@@
 	)
 	(junction
-		(at 275.59 25.4)
-		(diameter 0)
-		(color 0 0 0 0)
-	)
-	(junction
 		(at 87.63 26.67)
 		(diameter 0)
@@
 	)
 	(junction
+		(at 213.36 24.13)
+		(diameter 0)
+		(color 0 0 0 0)
+	)
+	(junction
 		(at 109.22 66.04)
 		(diameter 0)
@@
 	)
 	(junction
+		(at 275.59 25.4)
+		(diameter 0)
+		(color 0 0 0 0)
+	)
+	(junction
 		(at 138.43 50.8)
 		(diameter 0)
@@
 			)
 		)
-		(property "Footprint" "Connector_PinHeader_2.54mm:PinHeader_2x08_P2.54mm_Vertical"
+		(property "Footprint" "Connector_PinSocket_2.54mm:PinSocket_2x08_P2.54mm_Vertical"
 			(at 231.14 111.76 0)
 			(hide yes)
@@
 	)
 	(symbol
+		(lib_id "power:+5V")
+		(at 213.36 24.13 0)
+		(unit 1)
+		(body_style 1)
+		(exclude_from_sim no)
+		(in_bom yes)
+		(on_board yes)
+		(in_pos_files yes)
+		(dnp no)
+		(fields_autoplaced yes)
+		(property "Reference" "#PWR050"
+			(at 213.36 27.94 0)
+			(hide yes)
+			(show_name no)
+			(do_not_autoplace no)
+			(effects
+				(font
+					(size 1.27 1.27)
+				)
+			)
+		)
+		(property "Value" "+5V"
+			(at 213.36 19.05 0)
+			(show_name no)
+			(do_not_autoplace no)
+			(effects
+				(font
+					(size 1.27 1.27)
+				)
+			)
+		)
+		(property "Footprint" ""
+			(at 213.36 24.13 0)
+			(hide yes)
+			(show_name no)
+			(do_not_autoplace no)
+			(effects
+				(font
+					(size 1.27 1.27)
+				)
+			)
+		)
+		(property "Datasheet" ""
+			(at 213.36 24.13 0)
+			(hide yes)
+			(show_name no)
+			(do_not_autoplace no)
+			(effects
+				(font
+					(size 1.27 1.27)
+				)
+			)
+		)
+		(property "Description" "Power symbol creates a global label with name \"+5V\""
+			(at 213.36 24.13 0)
+			(hide yes)
+			(show_name no)
+			(do_not_autoplace no)
+			(effects
+				(font
+					(size 1.27 1.27)
+				)
+			)
+		)
+		(pin "1"
+		)
+		(instances
+			(project "mouth"
+				(path "/43a36e01-9c03-487f-b76f-d3e0c5ffafba"
+					(reference "#PWR050")
+					(unit 1)
+				)
+			)
+		)
+	)
+	(symbol
 		(lib_id "power:GND")
 		(at 52.07 99.06 0)
@@
 	)
 	(symbol
-		(lib_id "power:+3.3V")
+		(lib_id "power:+5V")
 		(at 275.59 25.4 0)
 		(unit 1)
@@
 		(dnp no)
 		(fields_autoplaced yes)
-		(property "Reference" "#PWR033"
+		(property "Reference" "#PWR051"
 			(at 275.59 29.21 0)
 			(hide yes)
@@
 			)
 		)
-		(property "Value" "+3.3V"
+		(property "Value" "+5V"
 			(at 275.59 20.32 0)
 			(show_name no)
@@
 			)
 		)
-		(property "Description" "Power symbol creates a global label with name \"+3.3V\""
+		(property "Description" "Power symbol creates a global label with name \"+5V\""
 			(at 275.59 25.4 0)
 			(hide yes)
@@
 			(project "mouth"
 				(path "/43a36e01-9c03-487f-b76f-d3e0c5ffafba"
-					(reference "#PWR033")
+					(reference "#PWR051")
 					(unit 1)
 				)
@@
 					(unit 1)
 				)
-			)
-		)
-	)
-	(symbol
-		(lib_id "power:+3.3V")
-		(at 213.36 24.13 0)
-		(unit 1)
-		(body_style 1)
-		(exclude_from_sim no)
-		(in_bom yes)
-		(on_board yes)
-		(in_pos_files yes)
-		(dnp no)
-		(fields_autoplaced yes)
-		(property "Reference" "#PWR020"
-			(at 213.36 27.94 0)
-			(hide yes)
-			(show_name no)
-			(do_not_autoplace no)
-			(effects
-				(font
-					(size 1.27 1.27)
-				)
-			)
-		)
-		(property "Value" "+3.3V"
-			(at 213.36 19.05 0)
-			(show_name no)
-			(do_not_autoplace no)
-			(effects
-				(font
-					(size 1.27 1.27)
-				)
-			)
-		)
-		(property "Footprint" ""
-			(at 213.36 24.13 0)
-			(hide yes)
-			(show_name no)
-			(do_not_autoplace no)
-			(effects
-				(font
-					(size 1.27 1.27)
-				)
-			)
-		)
-		(property "Datasheet" ""
-			(at 213.36 24.13 0)
-			(hide yes)
-			(show_name no)
-			(do_not_autoplace no)
-			(effects
-				(font
-					(size 1.27 1.27)
-				)
-			)
-		)
-		(property "Description" "Power symbol creates a global label with name \"+3.3V\""
-			(at 213.36 24.13 0)
-			(hide yes)
-			(show_name no)
-			(do_not_autoplace no)
-			(effects
-				(font
-					(size 1.27 1.27)
-				)
-			)
-		)
-		(pin "1"
-		)
-		(instances
-			(project "mouth"
-				(path "/43a36e01-9c03-487f-b76f-d3e0c5ffafba"
-					(reference "#PWR020")
-					(unit 1)
-				)

Commit message: more pcb
Connections:
- no-connect marks 12 -> 15
Changed lines of the file:
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@@
+	)
+	(no_connect
+		(at 124.46 124.46)
+	)
+	(no_connect
+		(at 124.46 127)
 	)
 	(no_connect
@@
 	)
 	(no_connect
+		(at 124.46 129.54)
+	)
+	(no_connect

Commit message: mostly do power part
Parts:
- J1: LCSC Part (none) -> C474881
- J5: LCSC Part (none) -> C30734
Changed lines of the file:
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@@
 			)
 		)
+		(property "LCSC Part" "C30734"
+			(at 231.14 111.76 0)
+			(hide yes)
+			(show_name no)
+			(do_not_autoplace no)
+			(effects
+				(font
+					(size 1.27 1.27)
+				)
+			)
+		)
 		(pin "13"
 		)
@@
 			(at 193.04 102.87 0)
 			(hide yes)
+			(show_name no)
+			(do_not_autoplace no)
+			(effects
+				(font
+					(size 1.27 1.27)
+				)
+			)
+		)
+		(property "LCSC Part" "C474881"
+			(at 193.04 102.87 0)
+			(hide yes)
