File: PCB/brain/_autosave-brain.kicad_sch (KiCad schematic)
At the start: 108 parts, among them J1 Screw_Terminal_01x02, J2 Conn_01x04, Q1 CSD17577Q3A, Q2 CSD17577Q3A, U1 ESP32-S3-WROOM-1, U10 MAX17049G+T10, U11 AP64501SP-13, U2 TMC2209-LA, U3 W5500, U4 MAX98357A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

Commit message: mostly do power part
Parts:
- added R27: 115k, Resistor_SMD:R_0603_1608Metric, symbol Device:R
- added R28: 22.1k, Resistor_SMD:R_0603_1608Metric, symbol Device:R
- L2: value L -> 3.6uH
Connections:
- net at L2.2: now also R27.1
- net at U11.5 (FB): now also R27.2, R28.1
Changed lines of the file:
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@@
 	)
 	(junction
+		(at 148.59 222.25)
+		(diameter 0)
+		(color 0 0 0 0)
+	)
+	(junction
 		(at 293.37 336.55)
 		(diameter 0)
@@
 	(wire
 		(pts
+			(xy 146.05 214.63) (xy 148.59 214.63)
+		)
+		(stroke
+			(width 0)
+			(type default)
+		)
+	)
+	(wire
+		(pts
 			(xy 204.47 31.75) (xy 213.36 31.75)
 		)
@@
 	(wire
 		(pts
+			(xy 118.11 222.25) (xy 148.59 222.25)
+		)
+		(stroke
+			(width 0)
+			(type default)
+		)
+	)
+	(wire
+		(pts
 			(xy 275.59 261.62) (xy 287.02 261.62)
 		)
@@
 	(wire
 		(pts
+			(xy 142.24 218.44) (xy 146.05 218.44)
+		)
+		(stroke
+			(width 0)
+			(type default)
+		)
+	)
+	(wire
+		(pts
 			(xy 266.7 363.22) (xy 266.7 364.49)
 		)
@@
 	(wire
 		(pts
+			(xy 146.05 218.44) (xy 146.05 214.63)
+		)
+		(stroke
+			(width 0)
+			(type default)
+		)
+	)
+	(wire
+		(pts
 			(xy 179.07 328.93) (xy 190.5 328.93)
 		)
@@
 	(symbol
 		(lib_id "Device:R")
+		(at 148.59 226.06 0)
+		(unit 1)
+		(body_style 1)
+		(exclude_from_sim no)
+		(in_bom yes)
+		(on_board yes)
+		(in_pos_files yes)
+		(dnp no)
+		(property "Reference" "R28"
+			(at 152.4 224.79 0)
+			(show_name no)
+			(do_not_autoplace no)
+			(effects
+				(font
+					(size 1.27 1.27)
+				)
+			)
+		)
+		(property "Value" "22.1k"
+			(at 153.162 227.33 0)
+			(show_name no)
+			(do_not_autoplace no)
+			(effects
+				(font
+					(size 1.27 1.27)
+				)
+			)
+		)
+		(property "Footprint" "Resistor_SMD:R_0603_1608Metric"
+			(at 146.812 226.06 90)
+			(hide yes)
+			(show_name no)
+			(do_not_autoplace no)
+			(effects
+				(font
+					(size 1.27 1.27)
+				)
+			)
+		)
+		(property "Datasheet" ""
+			(at 148.59 226.06 0)
+			(hide yes)
+			(show_name no)
+			(do_not_autoplace no)
+			(effects
+				(font
+					(size 1.27 1.27)
+				)
+			)
+		)
+		(property "Description" "Resistor"
+			(at 148.59 226.06 0)
+			(hide yes)
+			(show_name no)
+			(do_not_autoplace no)
+			(effects
+				(font
+					(size 1.27 1.27)
+				)
+			)
+		)
+		(pin "2"
+		)
+		(pin "1"
+		)
+		(instances
+			(project "brain"
+				(path "/83b42239-7ff5-41d9-ae38-aa795807f572"
+					(reference "R28")
+					(unit 1)
+				)
+			)
+		)
+	)
+	(symbol
+		(lib_id "Device:R")
 		(at 271.78 276.86 90)
 		(unit 1)
@@
 			)
 		)
-		(property "Value" "L"
+		(property "Value" "3.6uH"
 			(at 138.43 215.9 90)
 			(show_name no)
@@
 					(unit 1)
 				)
+			)
+		)
+	)
+	(symbol
+		(lib_id "Device:R")
+		(at 148.59 218.44 0)
+		(unit 1)
+		(body_style 1)
+		(exclude_from_sim no)
+		(in_bom yes)
+		(on_board yes)
+		(in_pos_files yes)
+		(dnp no)
+		(property "Reference" "R27"
+			(at 152.4 217.17 0)
+			(show_name no)
+			(do_not_autoplace no)
+			(effects
+				(font
+					(size 1.27 1.27)
+				)
+			)
+		)
+		(property "Value" "115k"
+			(at 153.162 219.71 0)
+			(show_name no)
+			(do_not_autoplace no)
+			(effects
+				(font
+					(size 1.27 1.27)
+				)
+			)
+		)
+		(property "Footprint" "Resistor_SMD:R_0603_1608Metric"
+			(at 146.812 218.44 90)
+			(hide yes)
+			(show_name no)
+			(do_not_autoplace no)
+			(effects
+				(font
+					(size 1.27 1.27)
+				)
+			)
+		)
+		(property "Datasheet" ""
+			(at 148.59 218.44 0)
+			(hide yes)
+			(show_name no)
+			(do_not_autoplace no)
+			(effects
+				(font
+					(size 1.27 1.27)
+				)
+			)
+		)
+		(property "Description" "Resistor"
+			(at 148.59 218.44 0)
+			(hide yes)
+			(show_name no)
+			(do_not_autoplace no)
+			(effects
+				(font
+					(size 1.27 1.27)
+				)
+			)
+		)
+		(pin "2"
+		)
+		(pin "1"
+		)
+		(instances
+			(project "brain"
+				(path "/83b42239-7ff5-41d9-ae38-aa795807f572"
+					(reference "R27")
+					(unit 1)
+				)
