File: PCB/brain/brain.kicad_pcb (KiCad board)
At the start: 4 copper layers, 100 x 115 mm, 223 parts, among them J1 Screw_Terminal_01x02, J10 Conn_01x12, J11 Conn_01x04, J12 BAT, J13 Conn_01x05, J14 Conn_01x02, J2 Conn_01x04, J3 RJ45_Hanrun_HR911105A_Horizon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, J4 Conn_01x04, J5 Conn_01x04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

Commit message: more pcb
Parts:
- added R60: 22R, Capacitor_SMD:C_0402_1005Metric, F.Cu at (96.1, 134.4)
- added R61: 22R, Capacitor_SMD:C_0402_1005Metric, F.Cu at (97.1, 134.4)
- moved R12 1.25 mm to (94.7, 136.7), turned to -90 degrees
Connections:
- U5 pad 1: D- -> DN
- U5 pad 2: D+ -> DP
- USB1 pad 5: D- -> DN
- USB1 pad 6: D+ -> DP
- USB1 pad 7: D- -> DN
- USB1 pad 8: D+ -> DP
Routing:
- net D-: track 15.7 -> 1.74 mm
- net DN: track 0.00 -> 12.9 mm
- net D+: track 14.3 -> 1.76 mm
- net DP: track 0.00 -> 12.3 mm
- net VUSB: track 6.85 -> 9.44 mm, vias 0 -> 4
- net GND: track 403.9 -> 402.7 mm, vias 216 -> 202
- added copper zone on B.Cu, net VUSB
- added copper zone on F.Cu, net VUSB
- added copper zone on In2.Cu, net VUSB

Commit message: DRC
Routing:
- net +3.3V: track 238.6 -> 246.9 mm
- net VBUS: track 37.5 -> 30.8 mm
- net Net-(U9-BTST1): track 2.61 -> 3.15 mm
- net GND: track 402.7 -> 402.9 mm, vias 202 -> 204

Commit message: more DRC
Routing:
- net GND: vias 204 -> 218
Changed lines of the file:
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@@
 		(tags "capacitor")
 		(property "Reference" "C45"
-			(at 0 -1.43 0)
+			(at 2.975 -0.025 0)
 			(layer "F.SilkS")
 			(effects
@@
 		(tags "capacitor")
 		(property "Reference" "C16"
-			(at 2.975 0 0)
+			(at 2.95 0.15 0)
 			(layer "F.SilkS")
 			(effects
@@
 		(descr "1.0uH ±20%")
 		(property "Reference" "L1"
-			(at 0 -4 90)
+			(at -0.01 -4.275 90)
 			(layer "F.SilkS")
 			(effects
@@
 		(tags "LED")
 		(property "Reference" "D4"
-			(at -2.6 0.05 90)
+			(at 2.39 -0.7 90)
 			(layer "F.SilkS")
 			(effects
@@
 		(tags "capacitor")
 		(property "Reference" "R61"
-			(at 0 1.545 90)
+			(at -2.675 0.6 90)
 			(layer "F.SilkS")
 			(effects
@@
 		(tags "2.4 GHz Wi-Fi and Bluetooth module")
 		(property "Reference" "U1"
-			(at -10.5 8.25 180)
+			(at -12.325 -0.11 180)
 			(unlocked yes)
 			(layer "F.SilkS")
@@
 		(tags "capacitor")
 		(property "Reference" "R60"
-			(at 0 -1.16 90)
+			(at -2.925 0.2 90)
 			(layer "F.SilkS")
 			(effects
@@
 		(tags "test point SMD pad")
 		(property "Reference" "TP3"
-			(at 0 -1.648 90)
+			(at -0.835 -2.175 90)
 			(layer "F.SilkS")
 			(effects
@@
 	)
 	(via
+		(at 100.875 138.3)
+		(size 0.5)
+		(drill 0.3)
+		(layers "F.Cu" "B.Cu")
+		(free yes)
+		(net "GND")
+	)
+	(via
 		(at 78 82)
 		(size 0.5)
@@
 	)
 	(via
+		(at 95.725 135.85)
+		(size 0.5)
+		(drill 0.3)
+		(layers "F.Cu" "B.Cu")
+		(free yes)
+		(net "GND")
+	)
+	(via
 		(at 98 99)
 		(size 0.5)
@@
 	)
 	(via
+		(at 96.6 137.5)
+		(size 0.5)
+		(drill 0.3)
+		(layers "F.Cu" "B.Cu")
+		(free yes)
+		(net "GND")
+	)
+	(via
 		(at 75 37.5)
 		(size 0.5)
@@
 	)
 	(via
+		(at 97.05 138.1)
+		(size 0.5)
+		(drill 0.3)
+		(layers "F.Cu" "B.Cu")
+		(free yes)
+		(net "GND")
+	)
+	(via
 		(at 142 76)
 		(size 0.5)
@@
 	)
 	(via
+		(at 98.15 135.375)
+		(size 0.5)
+		(drill 0.3)
+		(layers "F.Cu" "B.Cu")
+		(free yes)
+		(net "GND")
+	)
+	(via
+		(at 99.775 136.9)
+		(size 0.5)
+		(drill 0.3)
+		(layers "F.Cu" "B.Cu")
+		(free yes)
+		(net "GND")
+	)
+	(via
 		(at 85.75 125.25)
 		(size 0.5)
@@
 	)
 	(via
+		(at 101.35 138.875)
+		(size 0.5)
+		(drill 0.3)
+		(layers "F.Cu" "B.Cu")
+		(free yes)
+		(net "GND")
+	)
+	(via
 		(at 52.5 80)
 		(size 0.5)
@@
 	)
 	(via
+		(at 100.4 137.675)
+		(size 0.5)
+		(drill 0.3)
+		(layers "F.Cu" "B.Cu")
+		(free yes)
+		(net "GND")
+	)
+	(via
 		(at 133.2 122.4)
 		(size 0.5)
@@
 	)
 	(via
+		(at 98.775 135.925)
+		(size 0.5)
+		(drill 0.3)
+		(layers "F.Cu" "B.Cu")
+		(free yes)
+		(net "GND")
+	)
+	(via
 		(at 75.9 64.61)
 		(size 0.5)
@@
 	)
 	(via
+		(at 99.325 136.475)
+		(size 0.5)
+		(drill 0.3)
+		(layers "F.Cu" "B.Cu")
+		(free yes)
+		(net "GND")
+	)
+	(via
 		(at 81.85 81.65)
 		(size 0.5)
@@
 	)
 	(via
+		(at 97.7 138.7)
+		(size 0.5)
+		(drill 0.3)
+		(layers "F.Cu" "B.Cu")
+		(free yes)
+		(net "GND")
+	)
+	(via
 		(at 89 128)
 		(size 0.5)
@@
 	)
 	(via
+		(at 98.15 139.2)
+		(size 0.5)
+		(drill 0.3)
+		(layers "F.Cu" "B.Cu")
+		(free yes)
+		(net "GND")
+	)
+	(via
 		(at 72.5 37.5)
 		(size 0.5)
@@
 	)
 	(via
+		(at 101.85 139.275)
+		(size 0.5)
+		(drill 0.3)
+		(layers "F.Cu" "B.Cu")
+		(free yes)
+		(net "GND")
+	)
+	(via
 		(at 69 56)
 		(size 0.5)
@@
 	)
 	(via
+		(at 95.925 136.775)
+		(size 0.5)
+		(drill 0.3)
+		(layers "F.Cu" "B.Cu")
+		(free yes)
+		(net "GND")
+	)
+	(via
 		(at 66 61)
 		(size 0.5)
@@
 		(polygon
 			(pts
-				(xy 81 65.9225) (xy 81 64.7225) (xy 81.8 64.7225) (xy 82 64.9225) (xy 82 65.6225) (xy 82.1 65.7225)
+				(xy 80.95 65.9225) (xy 80.95 64.7225) (xy 81.8 64.7225) (xy 82 64.9225) (xy 82 65.6225) (xy 82.1 65.7225)
 				(xy 82.1 65.9225)
 			)
@@
 		(polygon
 			(pts
-				(xy 81.003768 66.525) (xy 81.003768 67.725) (xy 81.803768 67.725) (xy 82.003768 67.525) (xy 82.003768 66.825)
+				(xy 80.975 66.525) (xy 80.975 67.725) (xy 81.803768 67.725) (xy 82.003768 67.525) (xy 82.003768 66.825)
 				(xy 82.103768 66.725) (xy 82.103768 66.525)
 			)
